File: hardware/InterruptExpanderPCB/InterruptExpanderPCB/InterruptExpanderPCB.kicad_pcb (KiCad board)
At the start: 2 copper layers, 68.6 x 53.3 mm, 8 parts, among them J1 Power, J2 Digital/PWM, J3 Analog, J4 Digital/PWM

Commit message: working on tests
Parts:
- removed J4: Digital/PWM, Connector_PinSocket_2.54mm:PinSocket_1x08_P2.54mm_Vertical
- removed MH1, MH2, MH3, MH4: MountingHole_3.2mm, Arduino_MountingHole:MountingHole_3.2mm
- added C1: 0.1 uf, Capacitor_SMD:C_0402_1005Metric, F.Cu at (148.4, 57.5)
- added C10: 0.1 uf, Capacitor_SMD:C_0402_1005Metric, F.Cu at (151.3, 59.4)
- added C11: 0.1 uf, Capacitor_SMD:C_0402_1005Metric, F.Cu at (151.3, 61.4)
- added C12: 0.1 uf, Capacitor_SMD:C_0402_1005Metric, F.Cu at (151.3, 63.4)
- added C13: 0.1uf, Capacitor_SMD:C_0402_1005Metric, F.Cu at (151.3, 65.3)
- added C14: 1 uf, Capacitor_SMD:C_0603_1608Metric, F.Cu at (155.2, 73.5)
- added C2: 0.1uf, Capacitor_SMD:C_0402_1005Metric, F.Cu at (148.4, 59.4)
- added C3: 0.1uf, Capacitor_SMD:C_0402_1005Metric, F.Cu at (148.4, 61.4)
- added C4: 0.1uf, Capacitor_SMD:C_0402_1005Metric, F.Cu at (148.4, 63.4)
- added C5: 0.1 uf, Capacitor_SMD:C_0402_1005Metric, F.Cu at (148.4, 65.3)
- added C6: 0.1 uf, Capacitor_SMD:C_0402_1005Metric, F.Cu at (148.4, 67.3)
- added C7: 0.1 uf, Capacitor_SMD:C_0402_1005Metric, F.Cu at (148.4, 69.3)
- added C8: 0.1 uf, Capacitor_SMD:C_0402_1005Metric, F.Cu at (148.4, 71.2)
- added C9: 0.1 uf, Capacitor_SMD:C_0402_1005Metric, F.Cu at (151.3, 57.5)
- added D1: D_Zener, Diode_SMD:D_SOD-123, F.Cu at (155.3, 80.0)
- added D2: D, InterrupterLibrary:RF01128, F.Cu at (119.0, 35.4)
- added D3: D, InterrupterLibrary:RF01128, F.Cu at (119.0, 39.0)
- added R1: 10k, Capacitor_SMD:C_0402_1005Metric, F.Cu at (151.3, 67.3)
- added R10: 620, Capacitor_SMD:C_0402_1005Metric, F.Cu at (154.2, 69.3)
- added R11: 10k, Capacitor_SMD:C_0402_1005Metric, F.Cu at (154.2, 71.2)
- added R12: 620, Capacitor_SMD:C_0402_1005Metric, F.Cu at (157.0, 57.5)
- added R13: 10k, Capacitor_SMD:C_0402_1005Metric, F.Cu at (157.0, 59.4)
- added R14: 620, Capacitor_SMD:C_0402_1005Metric, F.Cu at (157.0, 61.4)
- added R15: 10k, Capacitor_SMD:C_0402_1005Metric, F.Cu at (157.0, 63.4)
- added R16: 620, Capacitor_SMD:C_0402_1005Metric, F.Cu at (157.0, 65.3)
- added R17: 10k, Capacitor_SMD:C_0402_1005Metric, F.Cu at (116.8, 41.8)
- added R2: 620, Capacitor_SMD:C_0402_1005Metric, F.Cu at (151.3, 69.3)
- added R3: 10k, Capacitor_SMD:C_0402_1005Metric, F.Cu at (151.3, 71.2)
- added R4: 620, Capacitor_SMD:C_0402_1005Metric, F.Cu at (154.2, 57.5)
- added R5: 10k, Capacitor_SMD:C_0402_1005Metric, F.Cu at (154.2, 59.4)
- added R6: 620, Capacitor_SMD:C_0402_1005Metric, F.Cu at (154.2, 61.4)
- added R7: 10k, Capacitor_SMD:C_0402_1005Metric, F.Cu at (154.2, 63.4)
- added R8: 620, Capacitor_SMD:C_0402_1005Metric, F.Cu at (154.2, 65.3)
- added R9: 10k, Capacitor_SMD:C_0402_1005Metric, F.Cu at (154.2, 67.3)
- added U1: ATTINY85-20SU, InterrupterLibrary:SOIC127P798X216-8N, F.Cu at (101.4, 43.4)
- added U2: SN74HC251PWR, InterrupterLibrary:SOP65P640X120-16N, F.Cu at (100.2, 50.1)
- added U3: SN74HC590ADT, InterrupterLibrary:SOIC127P600X175-16N, F.Cu at (117.5, 77.1)
- added U4: SN74HCT138PWRE4, InterrupterLibrary:SOP65P640X120-16N, F.Cu at (125.0, 63.5)
- J1: value Power -> Conn_01x06_Pin; footprint Connector_PinSocket_2.54mm:PinSocket_1x08_P2.54mm_Vertical -> Connector_PinHeader_2.00mm:PinHeader_1x06_P2.00mm_Vertical
- J2: value Digital/PWM -> Conn_01x08_Pin; footprint Connector_PinSocket_2.54mm:PinSocket_1x10_P2.54mm_Vertical -> Connector_PinHeader_2.00mm:PinHeader_1x08_P2.00mm_Vertical
- J3: value Analog -> Conn_01x08_Pin; footprint Connector_PinSocket_2.54mm:PinSocket_1x06_P2.54mm_Vertical -> Connector_PinHeader_2.00mm:PinHeader_1x08_P2.00mm_Vertical
- moved J1 50.8 mm to (160.5, 58.5), turned to 0 degrees
- moved J3 39.4 mm to (145.0, 58.5), turned to 0 degrees
- moved J2 27.0 mm to (136.0, 70.0), turned to 0 degrees
Connections:
- J1 pad 1: unconnected-(J1-Pin_1-Pad1) -> Net-(J1-Pin_1)
- J1 pad 2: /IOREF -> Net-(J1-Pin_2)
- J1 pad 3: /~{RESET} -> Net-(J1-Pin_3)
- J1 pad 4: +3V3 -> Net-(J1-Pin_4)
- J1 pad 5: +5V -> GND
- J1 pad 6: GND -> VCCQ
- J2 pad 1: /SCL/A5 -> Net-(J2-Pin_1)
- J2 pad 2: /SDA/A4 -> Net-(J2-Pin_2)
- J2 pad 3: /AREF -> Net-(J2-Pin_3)
- J2 pad 4: GND -> Net-(J2-Pin_4)
- J2 pad 5: /13 -> Net-(J2-Pin_5)
- J2 pad 6: /12 -> Net-(J2-Pin_6)
- J2 pad 7: /*11 -> Net-(J2-Pin_7)
- J2 pad 8: /*10 -> Net-(J2-Pin_8)
- J3 pad 1: /A0 -> Net-(J3-Pin_1)
- J3 pad 2: /A1 -> Net-(J3-Pin_2)
- J3 pad 3: /A2 -> Net-(J3-Pin_3)
- J3 pad 4: /A3 -> Net-(J3-Pin_4)
- J3 pad 5: /SDA/A4 -> Net-(J3-Pin_5)
- J3 pad 6: /SCL/A5 -> Net-(J3-Pin_6)
Other:
- board outline removed
- copper layers 2 -> 4
- board text removed: "ICSP"
